Commit message: 机械臂位数问题

File: evaluation/SoftFold-Agilex/Piper_ros_private-ros-noetic/src/piper_description/urdf/piper_description.urdf (robot description, URDF)
Before this commit: robot piper, 11 links, 10 joints
Links:
- link base_link: geometry collision mesh filename=/home/peng/x-vla-test/evaluation/SoftFold-Agilex/Piper_ros_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; visual mesh filename=/home/peng/x-vla-test/evaluation/SoftFold-Agilex/Piper_ros_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
- link gripper_base: geometry collision mesh filename=/home/peng/x-vla-test/evaluation/SoftFold-Agilex/Piper_ros_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; visual mesh filename=/home/peng/x-vla-test/evaluation/SoftFold-Agilex/Piper_ros_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
- link link1: geometry collision mesh filename=/home/peng/x-vla-test/evaluation/SoftFold-Agilex/Piper_ros_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; visual mesh filename=/home/peng/x-vla-test/evaluation/SoftFold-Agilex/Piper_ros_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
- link link2: geometry collision mesh filename=/home/peng/x-vla-test/evaluation/SoftFold-Agilex/Piper_ros_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; visual mesh filename=/home/peng/x-vla-test/evaluation/SoftFold-Agilex/Piper_ros_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
- link link3: geometry collision mesh filename=/home/peng/x-vla-test/evaluation/SoftFold-Agilex/Piper_ros_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; visual mesh filename=/home/peng/x-vla-test/evaluation/SoftFold-Agilex/Piper_ros_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
- link link4: geometry collision mesh filename=/home/peng/x-vla-test/evaluation/SoftFold-Agilex/Piper_ros_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; visual mesh filename=/home/peng/x-vla-test/evaluation/SoftFold-Agilex/Piper_ros_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
- link link5: geometry collision mesh filename=/home/peng/x-vla-test/evaluation/SoftFold-Agilex/Piper_ros_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; visual mesh filename=/home/peng/x-vla-test/evaluation/SoftFold-Agilex/Piper_ros_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
- link link6: geometry collision mesh filename=/home/peng/x-vla-test/evaluation/SoftFold-Agilex/Piper_ros_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; visual mesh filename=/home/peng/x-vla-test/evaluation/SoftFold-Agilex/Piper_ros_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
- link link7: geometry collision mesh filename=/home/peng/x-vla-test/evaluation/SoftFold-Agilex/Piper_ros_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; visual mesh filename=/home/peng/x-vla-test/evaluation/SoftFold-Agilex/Piper_ros_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
- link link8: geometry collision mesh filename=/home/peng/x-vla-test/evaluation/SoftFold-Agilex/Piper_ros_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; visual mesh filename=/home/peng/x-vla-test/evaluation/SoftFold-Agilex/Piper_ros_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

Commit message: 复用ik逻辑，重新梳理观测输入

File: evaluation/SoftFold-Agilex/Piper_ros_private-ros-noetic/src/piper_description/urdf/piper_description.urdf (robot description, URDF)
Before this commit: robot piper, 11 links, 10 joints
Links:
- link base_link: geometry collision mesh filename=/home/lyj/X-VLA/evaluation/SoftFold-Agilex/Piper_ros_privat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; visual mesh filename=/home/lyj/X-VLA/evaluation/SoftFold-Agilex/Piper_ros_privat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
- link gripper_base: geometry collision mesh filename=/home/lyj/X-VLA/evaluation/SoftFold-Agilex/Piper_ros_privat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; visual mesh filename=/home/lyj/X-VLA/evaluation/SoftFold-Agilex/Piper_ros_privat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
- link link1: geometry collision mesh filename=/home/lyj/X-VLA/evaluation/SoftFold-Agilex/Piper_ros_privat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; visual mesh filename=/home/lyj/X-VLA/evaluation/SoftFold-Agilex/Piper_ros_privat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
- link link2: geometry collision mesh filename=/home/lyj/X-VLA/evaluation/SoftFold-Agilex/Piper_ros_privat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; visual mesh filename=/home/lyj/X-VLA/evaluation/SoftFold-Agilex/Piper_ros_privat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
- link link3: geometry collision mesh filename=/home/lyj/X-VLA/evaluation/SoftFold-Agilex/Piper_ros_privat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; visual mesh filename=/home/lyj/X-VLA/evaluation/SoftFold-Agilex/Piper_ros_privat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
- link link4: geometry collision mesh filename=/home/lyj/X-VLA/evaluation/SoftFold-Agilex/Piper_ros_privat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; visual mesh filename=/home/lyj/X-VLA/evaluation/SoftFold-Agilex/Piper_ros_privat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
- link link5: geometry collision mesh filename=/home/lyj/X-VLA/evaluation/SoftFold-Agilex/Piper_ros_privat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; visual mesh filename=/home/lyj/X-VLA/evaluation/SoftFold-Agilex/Piper_ros_privat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
- link link6: geometry collision mesh filename=/home/lyj/X-VLA/evaluation/SoftFold-Agilex/Piper_ros_privat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; visual mesh filename=/home/lyj/X-VLA/evaluation/SoftFold-Agilex/Piper_ros_privat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
- link link7: geometry collision mesh filename=/home/lyj/X-VLA/evaluation/SoftFold-Agilex/Piper_ros_privat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; visual mesh filename=/home/lyj/X-VLA/evaluation/SoftFold-Agilex/Piper_ros_privat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
- link link8: geometry collision mesh filename=/home/lyj/X-VLA/evaluation/SoftFold-Agilex/Piper_ros_privat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; visual mesh filename=/home/lyj/X-VLA/evaluation/SoftFold-Agilex/Piper_ros_privat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
